File: Circuitos/Mixer 4 Channels with Power Amplifier/subnets/mixer_subnet/Preamplifier.kicad_sch (KiCad schematic)
At the start: 6 parts

Commit message: Correcciones en etapas y respaldo fotos simulación
Parts:
- Ci: value 8.2uF -> 2.2uF
- Rf?: value 33 -> 390
- Ri?: value 1k -> 3.9k
Changed lines of the file:
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@@
 			)
 		)
-		(property "Value" "8.2uF"
+		(property "Value" "2.2uF"
 			(at 114.681 87.63 90)
 			(effects
@@
 			)
 		)
-		(property "Value" "1k"
+		(property "Value" "3.9k"
 			(at 125.7299 90.17 90)
 			(effects
@@
 			)
 		)
-		(property "Value" "33"
+		(property "Value" "390"
 			(at 135.89 79.248 90)
 			(effects
