File: Circuitos/Mixer 4 Channels with Power Amplifier/subnets/mixer_subnet/VU Meter.kicad_sch (KiCad schematic)
At the start: 14 parts

Commit message: Correcciones y modificaciones en fuente, amp auriculares y simul completa
Parts:
- R_led?: value 680 -> 510
Changed lines of the file:
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@@
 			)
 		)
-		(property "Value" "680"
+		(property "Value" "510"
 			(at 165.0999 82.55 90)
 			(effects
