File: Circuitos/Mixer 4 Channels with Power Amplifier/subnets/mixer_subnet/Tone Control.kicad_sch (KiCad schematic)
At the start: 23 parts, among them U10 ${SIM.PARAMS}, U7 ${SIM.PARAMS}

Commit message: Final de proyecto
Connections:
- net at C6.1, R10.1, U10.2 (-): now also C5.2, R11.2
Changed lines of the file:
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@@
+	)
+	(junction
+		(at 166.37 123.19)
+		(diameter 0)
+		(color 0 0 0 0)
+	)
+	(junction
+		(at 166.37 102.87)
+		(diameter 0)
+		(color 0 0 0 0)
 	)
 	(junction
@@
 	(wire
 		(pts
+			(xy 166.37 123.19) (xy 182.88 123.19)
+		)
+		(stroke
+			(width 0)
+			(type default)
+		)
+	)
+	(wire
+		(pts
 			(xy 152.4 64.77) (xy 151.13 64.77)
 		)
@@
 	(wire
 		(pts
+			(xy 166.37 102.87) (xy 166.37 123.19)
+		)
+		(stroke
+			(width 0)
+			(type default)
+		)
+	)
+	(wire
+		(pts
 			(xy 109.22 76.2) (xy 115.57 76.2)
 		)
@@
 	(wire
 		(pts
-			(xy 156.21 123.19) (xy 182.88 123.19)
-		)
-		(stroke
+			(xy 156.21 123.19) (xy 166.37 123.19)
+		)
+		(stroke
