File: Circuitos/Mixer 4 Channels with Power Amplifier/subnets/Class AB Power Amplifier.kicad_sch (KiCad schematic)
At the start: 10 parts, among them Q1 TIP31C, Q2 TIP32C, Q3 2N3906, Q4 2N3904

Commit message: Correcciones y modificaciones en fuente, amp auriculares y simul completa
Parts:
- Q1: value TIP31C -> TIP31
- Q2: value TIP32C -> TIP32
- Rb1, Rb2: value 6.8k -> 4.7k
Changed lines of the file:
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@@
 			)
 		)
-		(property "Value" "6.8k"
+		(property "Value" "4.7k"
 			(at 130.81 70.358 0)
 			(effects
@@
 				)
 				(justify right)
+				(hide yes)
 			)
 		)
@@
 				)
 				(justify right)
+				(hide yes)
 			)
 		)
@@
 			)
 		)
-		(property "Value" "TIP32C"
+		(property "Value" "TIP32"
 			(at 161.29 68.5801 0)
 			(effects
@@
 			)
 		)
-		(property "Value" "TIP31C"
+		(property "Value" "TIP31"
 			(at 161.29 118.1099 0)
 			(effects
@@
 			)
 		)
-		(property "Value" "6.8k"
+		(property "Value" "4.7k"
 			(at 130.81 118.872 0)
 			(effects
