File: Circuitos/Mixer 4 Channels with Power Amplifier/Mixer 4 Channels with Power Amplifier.kicad_sch (KiCad schematic)
At the start: 4 parts

Commit message: Informe finalizado
Other:
- added sheet Regulador2 (subnets/Regulador.kicad_sch)
