File: Circuitos/Fuente de Alimentación/Fuente de Alimentación.kicad_sch (KiCad schematic)
At the start: 24 parts, among them Q1 NPN, Q2 PNP, Q3 PNP, Q4 NPN, T1 Transformer_1P_SS, U1 LM7815_TO220, U3 LM7915_TO220

Commit message: Power Supply corrections
Connections:
- net -Power: now also Q4.3 (E); no longer Q4.1 (C)
- net -V: now also Q1.1 (C); no longer Q1.3 (E)
- net at C4.2, Q4.2 (B), R5.2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: now also Q1.3 (E); no longer Q1.1 (C)
- net at Q1.2 (B), R6.2: now also Q4.1 (C); no longer Q4.3 (E)
Other:
- moved on the sheet: Q1, Q4
Changed lines of the file:
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@@
 (kicad_sch
-	(version 20231120)
+	(version 20250114)
 	(generator "eeschema")
-	(generator_version "8.0")
+	(generator_version "9.0")
 	(paper "A4")
 	(junction
@@
 	(symbol
 		(lib_id "Simulation_SPICE:NPN")
-		(at 87.63 151.13 270)
+		(at 87.63 151.13 90)
+		(mirror x)
 		(unit 1)
 		(exclude_from_sim no)
@@
 	(symbol
 		(lib_id "Simulation_SPICE:NPN")
-		(at 80.01 148.59 270)
-		(mirror x)
+		(at 80.01 148.59 90)
 		(unit 1)
 		(exclude_from_sim no)
@@
 		)
 	)
+	(embedded_fonts no)
 )
